File: Mega Breakout.brd (EAGLE design)
At the start: 101.6 x 61.9 mm, 13 parts

Commit message: Finished PCB
Parts:
- moved PWM 1.27 mm to (24.1, 59.2)
- moved POWER 0.57 mm to (21.3, 10.7)
Routing:
- net AREF: track 0.00 -> 43.4 mm
- net RESET: track 32.0 -> 32.6 mm
- net +3V3: track 32.0 -> 32.6 mm
- net 2: track 33.5 -> 33.0 mm
- net 7: track 33.5 -> 33.0 mm
- net 6: track 33.5 -> 33.0 mm
- net 5: track 33.5 -> 33.0 mm
- net 4: track 33.5 -> 33.0 mm
- net 3: track 33.5 -> 33.0 mm
- net 13: track 37.8 -> 37.3 mm
- net 12: track 37.2 -> 36.7 mm
- net 11: track 36.6 -> 36.1 mm
- net 10: track 36.0 -> 35.4 mm
- net 9: track 35.3 -> 34.8 mm
- net 8: track 34.7 -> 34.1 mm
Other:
- board text added: "+5V CS1-47 DIR1-48 PUL1-49 MISO-50 MOSI-51 SCK-52 GND"
- board text added: "+5V CS2-44 DIR2-45 PUL2-46 MISO-50 MOSI-51 SCK-52 GND"
- board text added: "+5V CS3-41 DIR3-42 PUL3-43 MISO-50 MOSI-51 SCK-52 GND"
- board text added: "+5V CS4-38 DIR4-39 PUL4-40 MISO-50 MOSI-51 SCK-52 GND"
- board text added: "+5V CS5-35 DIR5-36 PUL5-37 MISO-50 MOSI-51 SCK-52 GND"
- board text added: "+5V CS6-32 DIR6-33 PUL6-34 MISO-50 MOSI-51 SCK-52 GND"
- board text removed: "+5V CS1-47 DIR1-48 PUL1-49 MISO-50"
- board text removed: "+5V CS2-44 DIR2-45 PUL2-46 MISO-50"
- board text removed: "+5V CS3-41 DIR3-42 PUL3-43 MISO-50"
- board text removed: "+5V CS4-38 DIR4-39 PUL4-40 MISO-50"
- board text removed: "+5V CS5-35 DIR5-36 PUL5-37 MISO-50"
- board text removed: "+5V CS6-32 DIR6-33"
- board text removed: "GND"
- board text removed: "MISO-50"
- board text removed: "MOSI-51"
- board text removed: "PUL6-34"
- board text removed: "SCK-52"
