File: Mega Breakout with more GNDs_final.brd (EAGLE design)
At the start: 101.6 x 61.9 mm, 13 parts

Commit message: final ver of modified PCB
Routing:
- net GND: track 159.8 -> 189.1 mm
Changed lines of the file:
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@@
 <wire x1="33.02" y1="48.768" x2="33.02" y2="50.8" width="0.1524" layer="16"/>
 <wire x1="30.3812" y1="40.58095" x2="30.3812" y2="46.1292" width="0.1524" layer="16"/>
-<wire x1="100.33" y1="7.62" x2="102.87" y2="7.62" width="0" layer="19" extent="1-1"/>
-<wire x1="87.376" y1="19.812" x2="100.33" y2="7.62" width="0" layer="19" extent="1-1"/>
-<wire x1="87.376" y1="22.352" x2="87.376" y2="19.812" width="0" layer="19" extent="1-1"/>
-<wire x1="87.376" y1="24.892" x2="87.376" y2="22.352" width="0" layer="19" extent="1-1"/>
+<wire x1="87.376" y1="24.892" x2="87.376" y2="22.352" width="0.1524" layer="1"/>
+<wire x1="87.376" y1="22.352" x2="87.376" y2="19.812" width="0.1524" layer="1"/>
+<wire x1="87.376" y1="19.812" x2="91.44" y2="15.748" width="0.1524" layer="1"/>
+<wire x1="91.44" y1="15.748" x2="91.44" y2="13.716" width="0.1524" layer="1"/>
+<wire x1="91.44" y1="13.716" x2="97.536" y2="7.62" width="0.1524" layer="1"/>
+<wire x1="97.536" y1="7.62" x2="100.33" y2="7.62" width="0.1524" layer="1"/>
+<wire x1="100.33" y1="7.62" x2="102.87" y2="7.62" width="0.1524" layer="1"/>
+<wire x1="46.99" y1="2.54" x2="49.53" y2="2.54" width="0.1524" layer="16"/>
 <wire x1="72.136" y1="19.812" x2="72.136" y2="22.352" width="0" layer="19" extent="1-1"/>
 <wire x1="72.136" y1="24.892" x2="72.136" y2="22.352" width="0" layer="19" extent="1-1"/>
 <wire x1="56.896" y1="22.352" x2="56.896" y2="24.892" width="0" layer="19" extent="1-1"/>
 <wire x1="56.896" y1="19.812" x2="56.896" y2="22.352" width="0" layer="19" extent="1-1"/>
-<wire x1="49.53" y1="2.54" x2="46.99" y2="2.54" width="0" layer="19" extent="1-1"/>
 <wire x1="25.146" y1="10.668" x2="27.686" y2="10.668" width="0" layer="19" extent="1-1"/>
 <wire x1="11.176" y1="22.352" x2="11.176" y2="19.812" width="0" layer="19" extent="1-1"/>
@@
 <wire x1="101.6" y1="21.59" x2="99.314" y2="21.59" width="0.1524" layer="16"/>
 <wire x1="99.314" y1="21.59" x2="94.488" y2="16.764" width="0.1524" layer="16"/>
-<wire x1="94.488" y1="16.764" x2="87.122" y2="16.764" width="0.1524" layer="16"/>
-<via x="87.122" y="16.764" extent="1-16" drill="0.35"/>
+<wire x1="94.488" y1="16.764" x2="86.868" y2="16.764" width="0.1524" layer="16"/>
+<via x="86.868" y="16.764" extent="1-16" drill="0.35"/>
 <via x="62.23" y="22.098" extent="1-16" drill="0.35"/>
-<wire x1="62.23" y1="29.718" x2="58.42" y2="33.528" width="0.1524" layer="16"/>
+<wire x1="62.23" y1="29.718" x2="56.896" y2="35.052" width="0.1524" layer="16"/>
 <wire x1="62.23" y1="22.098" x2="67.564" y2="16.764" width="0.1524" layer="1"/>
-<wire x1="67.564" y1="16.764" x2="87.122" y2="16.764" width="0.1524" layer="1"/>
+<wire x1="67.564" y1="16.764" x2="86.868" y2="16.764" width="0.1524" layer="1"/>
 <contactref element="JP3" pad="7"/>
-<wire x1="56.896" y1="35.052" x2="58.42" y2="33.528" width="0.1524" layer="16"/>
 <wire x1="62.23" y1="29.718" x2="62.23" y2="22.098" width="0.1524" layer="16"/>
 </signal>
@@
 <wire x1="84.836" y1="21.336" x2="92.71" y2="21.336" width="0.1524" layer="16"/>
 <wire x1="92.71" y1="21.336" x2="99.314" y2="27.94" width="0.1524" layer="16"/>
-<via x="75.184" y="19.304" extent="1-16" drill="0.35"/>
-<wire x1="74.295" y1="18.415" x2="75.184" y2="19.304" width="0.1524" layer="16"/>
-<wire x1="84.836" y1="21.336" x2="77.216" y2="21.336" width="0.1524" layer="1"/>
-<wire x1="77.216" y1="21.336" x2="75.184" y2="19.304" width="0.1524" layer="1"/>
+<via x="75.438" y="19.05" extent="1-16" drill="0.35"/>
+<wire x1="74.676" y1="18.288" x2="75.438" y2="19.05" width="0.1524" layer="16"/>
+<wire x1="84.836" y1="21.336" x2="77.724" y2="21.336" width="0.1524" layer="1"/>
+<wire x1="77.724" y1="21.336" x2="75.438" y2="19.05" width="0.1524" layer="1"/>
 <contactref element="JP4" pad="9"/>
 <wire x1="51.054" y1="30.734" x2="51.054" y2="19.304" width="0.1524" layer="16"/>
 <wire x1="51.054" y1="19.304" x2="52.07" y2="18.288" width="0.1524" layer="16"/>
-<wire x1="74.168" y1="18.288" x2="74.295" y2="18.415" width="0.1524" layer="16"/>
-<wire x1="52.07" y1="18.288" x2="74.168" y2="18.288" width="0.1524" layer="16"/>
+<wire x1="52.07" y1="18.288" x2="74.676" y2="18.288" width="0.1524" layer="16"/>
 </signal>
 <signal name="DIR4-39">
@@
 <wire x1="99.314" y1="26.67" x2="93.472" y2="20.828" width="0.1524" layer="16"/>
 <wire x1="93.472" y1="20.828" x2="93.46438125" y2="20.82038125" width="0.1524" layer="16"/>
-<wire x1="74.93" y1="17.272" x2="76.962" y2="19.304" width="0.1524" layer="16"/>
-<via x="76.962" y="19.304" extent="1-16" drill="0.35"/>
-<wire x1="76.962" y1="19.304" x2="76.9772375" y2="19.304" width="0.1524" layer="1"/>
-<via x="83.82761875" y="20.31238125" extent="1-16" drill="0.35"/>
+<wire x1="74.93" y1="17.272" x2="76.708" y2="19.05" width="0.1524" layer="16"/>
+<via x="76.708" y="19.05" extent="1-16" drill="0.35"/>
+<wire x1="76.708" y1="19.05" x2="76.7232375" y2="19.05" width="0.1524" layer="1"/>
+<via x="83.82761875" y="20.56638125" extent="1-16" drill="0.35"/>
 <contactref element="JP4" pad="8"/>
 <wire x1="50.292" y1="28.956" x2="50.292" y2="19.05" width="0.1524" layer="16"/>
 <wire x1="50.292" y1="19.05" x2="52.07" y2="17.272" width="0.1524" layer="16"/>
 <wire x1="52.07" y1="17.272" x2="74.93" y2="17.272" width="0.1524" layer="16"/>
-<wire x1="83.312" y1="20.828" x2="83.82761875" y2="20.31238125" width="0.1524" layer="1"/>
-<wire x1="76.9772375" y1="19.304" x2="78.5012375" y2="20.828" width="0.1524" layer="1"/>
-<wire x1="78.5012375" y1="20.828" x2="83.312" y2="20.828" width="0.1524" layer="1"/>
-<wire x1="83.82761875" y1="20.31238125" x2="84.0892375" y2="20.574" width="0.1524" layer="16"/>
+<wire x1="76.7232375" y1="19.05" x2="78.2472375" y2="20.574" width="0.1524" layer="1"/>
+<wire x1="83.82761875" y1="20.56638125" x2="83.8352375" y2="20.574" width="0.1524" layer="16"/>
 <wire x1="85.852" y1="20.574" x2="86.3092" y2="21.0312" width="0.1524" layer="16"/>
 <wire x1="88.6968" y1="21.0312" x2="88.9" y2="20.828" width="0.1524" layer="16"/>
 <wire x1="88.9" y1="20.828" x2="93.472" y2="20.828" width="0.1524" layer="16"/>
-<wire x1="84.0892375" y1="20.574" x2="85.852" y2="20.574" width="0.1524" layer="16"/>
+<wire x1="83.8352375" y1="20.574" x2="85.852" y2="20.574" width="0.1524" layer="16"/>
 <wire x1="86.3092" y1="21.0312" x2="88.6968" y2="21.0312" width="0.1524" layer="16"/>
+<wire x1="78.2472375" y1="20.574" x2="83.82" y2="20.574" width="0.1524" layer="1"/>
+<wire x1="83.82" y1="20.574" x2="83.82761875" y2="20.56638125" width="0.1524" layer="1"/>
 </signal>
 <signal name="PUL5-37">

Commit message: final ver of modified PCB
Routing:
- net GND: track 189.1 -> 22.1 mm, vias 0 -> 1

Commit message: final ver of modified PCB
Routing:
- net PUL5-37: track 84.9 -> 81.9 mm
- net DIR5-36: track 81.3 -> 78.3 mm
- net CS2-44: track 46.4 -> 48.3 mm
- net PUL3-43: track 60.5 -> 62.4 mm
- net GND: track 22.1 -> 20.3 mm, vias 1 -> 0
- net DIR2-45: track 47.9 -> 49.4 mm
- net 25: track 50.6 -> 52.0 mm, vias 0 -> 1
- net +5V: track 146.8 -> 145.5 mm
- net PUL2-46: track 43.3 -> 44.5 mm
- net DIR4-39: track 79.9 -> 80.7 mm
- net CS4-38: track 78.4 -> 79.3 mm
- net PUL4-40: track 75.4 -> 76.0 mm
